Commit message: Use robot namespace parameter

File: husky_description/urdf/accessories/intel_realsense.urdf.xacro (robot description, xacro)
@@ -1,5 +1,5 @@
 <?xml version="1.0"?>
 <robot xmlns:xacro="http://ros.org/wiki/xacro">
-  <xacro:macro name="intel_realsense_mount" params="prefix topic parent_link">
+  <xacro:macro name="intel_realsense_mount" params="prefix topic parent_link robot_namespace">
     <xacro:macro name="intel_realsense" params="
                frame:=realsense          topic:=realsense
@@ -8,5 +8,5 @@
                width:=640                height:=480
                update_rate:=30
-               robot_namespace:=/">
+               robot_namespace:=$(arg robot_namespace)">
       <!-- this link is the origin for the camera's data -->
       <link name="${frame}" />
@@ -46,5 +46,5 @@
             <alwaysOn>true</alwaysOn>
             <updateRate>${update_rate}</updateRate>
-            <cameraName>${topic}</cameraName>
+            <cameraName>${robot_namespace}/${topic}</cameraName>
             <imageTopicName>color/image_raw</imageTopicName>
             <cameraInfoTopicName>color/camera_info</cameraInfoTopicName>
@@ -52,5 +52,5 @@
             <depthImageInfoTopicName>depth/camera_info</depthImageInfoTopicName>
             <pointCloudTopicName>depth/color/points</pointCloudTopicName>
-            <frameName>husky/${frame}_gazebo</frameName>
+            <frameName>${robot_namespace}/${frame}_gazebo</frameName>
             <pointCloudCutoff>${min_range}</pointCloudCutoff>
             <pointCloudCutoffMax>${max_range}</pointCloudCutoffMax>

File: husky_description/urdf/husky.urdf.xacro (robot description, xacro)
@@ -144,5 +144,5 @@
       <child link="realsense_mountpoint" />
     </joint>
-    <xacro:intel_realsense_mount prefix="camera" topic="realsense" parent_link="realsense_mountpoint"/>
+    <xacro:intel_realsense_mount prefix="camera" topic="realsense" robot_namespace="$(arg robot_namespace)" parent_link="realsense_mountpoint"/>
   </xacro:if>
   <gazebo>

Commit message: xacro updates
* Updated xacro to use robot namespace

* Updated xacro such that depth image FOV corresponds to RGB image FOV

File: husky_description/urdf/accessories/intel_realsense.urdf.xacro (robot description, xacro)
@@ -1,12 +1,12 @@
 <?xml version="1.0"?>
 <robot xmlns:xacro="http://ros.org/wiki/xacro">
-  <xacro:macro name="intel_realsense_mount" params="prefix topic parent_link">
+  <xacro:macro name="intel_realsense_mount" params="prefix topic parent_link robot_namespace">
     <xacro:macro name="intel_realsense" params="
                frame:=realsense          topic:=realsense
-               h_fov:=1.5184351666666667 v_fov:=1.0122901111111111
+               h_fov:=1.5184351666666667 v_fov:=1.1388273
                min_range:=0.105          max_range:=8.0
                width:=640                height:=480
                update_rate:=30
-               robot_namespace:=/">
+               robot_namespace:=$(arg robot_namespace)">
       <!-- this link is the origin for the camera's data -->
       <link name="${frame}" />
@@ -46,5 +46,5 @@
             <alwaysOn>true</alwaysOn>
             <updateRate>${update_rate}</updateRate>
-            <cameraName>${topic}</cameraName>
+            <cameraName>${robot_namespace}/${topic}</cameraName>
             <imageTopicName>color/image_raw</imageTopicName>
             <cameraInfoTopicName>color/camera_info</cameraInfoTopicName>
@@ -52,5 +52,5 @@
             <depthImageInfoTopicName>depth/camera_info</depthImageInfoTopicName>
             <pointCloudTopicName>depth/color/points</pointCloudTopicName>
-            <frameName>${frame}_gazebo</frameName>
+            <frameName>${robot_namespace}/${frame}_gazebo</frameName>
             <pointCloudCutoff>${min_range}</pointCloudCutoff>
             <pointCloudCutoffMax>${max_range}</pointCloudCutoffMax>

File: husky_description/urdf/husky.urdf.xacro (robot description, xacro)
@@ -168,5 +168,5 @@
       <child link="realsense_mountpoint" />
     </joint>
-    <xacro:intel_realsense_mount prefix="camera" topic="realsense" parent_link="realsense_mountpoint"/>
+    <xacro:intel_realsense_mount prefix="camera" topic="realsense" robot_namespace="$(arg robot_namespace)" parent_link="realsense_mountpoint"/>
   </xacro:if>
   <!--

Commit message: Added use_namespace to husky xacro

File: husky_description/urdf/accessories/intel_realsense.urdf.xacro (robot description, xacro)
@@ -1,5 +1,5 @@
 <?xml version="1.0"?>
 <robot xmlns:xacro="http://ros.org/wiki/xacro">
-  <xacro:macro name="intel_realsense_mount" params="prefix topic parent_link robot_namespace">
+  <xacro:macro name="intel_realsense_mount" params="prefix topic parent_link use_namespace robot_namespace">
     <xacro:macro name="intel_realsense" params="
                frame:=realsense          topic:=realsense
@@ -8,4 +8,5 @@
                width:=640                height:=480
                update_rate:=30
+               use_namespace:=$(arg use_namespace)
                robot_namespace:=$(arg robot_namespace)">
       <!-- this link is the origin for the camera's data -->
@@ -52,5 +53,10 @@
             <depthImageInfoTopicName>depth/camera_info</depthImageInfoTopicName>
             <pointCloudTopicName>depth/color/points</pointCloudTopicName>
-            <frameName>${robot_namespace}/${frame}_gazebo</frameName>
+            <xacro:if value="${use_namespace}">
+              <frameName>${robot_namespace}/${frame}_gazebo</frameName>
+            </xacro:if>
+            <xacro:unless value="${use_namespace}">
+              <frameName>${frame}_gazebo</frameName>
+            </xacro:unless>
             <pointCloudCutoff>${min_range}</pointCloudCutoff>
             <pointCloudCutoffMax>${max_range}</pointCloudCutoffMax>

File: husky_description/urdf/husky.urdf.xacro (robot description, xacro)
@@ -40,4 +40,5 @@
   <xacro:arg name="sensor_arch_height"  default="$(optenv HUSKY_SENSOR_ARCH_HEIGHT 510)" />
   <xacro:arg name="sensor_arch"         default="$(optenv HUSKY_SENSOR_ARCH 0)" />
+  <xacro:arg name="use_namespace" default="$(optenv USE_NAMESPACE false)" />
   <xacro:arg name="robot_namespace" default="$(optenv ROBOT_NAMESPACE /)" />
   <xacro:arg name="urdf_extras" default="$(optenv HUSKY_URDF_EXTRAS empty.urdf)" />
@@ -168,5 +169,5 @@
       <child link="realsense_mountpoint" />
     </joint>
-    <xacro:intel_realsense_mount prefix="camera" topic="realsense" robot_namespace="$(arg robot_namespace)" parent_link="realsense_mountpoint"/>
+    <xacro:intel_realsense_mount prefix="camera" topic="realsense" use_namespace="$(arg use_namespace)" robot_namespace="$(arg robot_namespace)" parent_link="realsense_mountpoint"/>
   </xacro:if>
   <!--

Commit message: fixing some redundant ns issues

File: husky_description/urdf/accessories/intel_realsense.urdf.xacro (robot description, xacro)
@@ -1,5 +1,5 @@
 <?xml version="1.0"?>
 <robot xmlns:xacro="http://ros.org/wiki/xacro">
-  <xacro:macro name="intel_realsense_mount" params="prefix topic parent_link use_namespace robot_namespace">
+  <xacro:macro name="intel_realsense_mount" params="prefix topic parent_link robot_namespace">
     <xacro:macro name="intel_realsense" params="
                frame:=realsense          topic:=realsense
@@ -8,5 +8,4 @@
                width:=640                height:=480
                update_rate:=30
-               use_namespace:=$(arg use_namespace)
                robot_namespace:=$(arg robot_namespace)">
       <!-- this link is the origin for the camera's data -->
@@ -47,5 +46,5 @@
             <alwaysOn>true</alwaysOn>
             <updateRate>${update_rate}</updateRate>
-            <cameraName>${robot_namespace}/${topic}</cameraName>
+            <cameraName>${topic}</cameraName>
             <imageTopicName>color/image_raw</imageTopicName>
             <cameraInfoTopicName>color/camera_info</cameraInfoTopicName>
@@ -53,10 +52,5 @@
             <depthImageInfoTopicName>depth/camera_info</depthImageInfoTopicName>
             <pointCloudTopicName>depth/color/points</pointCloudTopicName>
-            <xacro:if value="${use_namespace}">
-              <frameName>${robot_namespace}/${frame}_gazebo</frameName>
-            </xacro:if>
-            <xacro:unless value="${use_namespace}">
-              <frameName>${frame}_gazebo</frameName>
-            </xacro:unless>
+            <frameName>${robot_namespace}/${frame}_gazebo</frameName>
             <pointCloudCutoff>${min_range}</pointCloudCutoff>
             <pointCloudCutoffMax>${max_range}</pointCloudCutoffMax>

File: husky_description/urdf/husky.urdf.xacro (robot description, xacro)
@@ -169,5 +169,5 @@
       <child link="realsense_mountpoint" />
     </joint>
-    <xacro:intel_realsense_mount prefix="camera" topic="realsense" use_namespace="$(arg use_namespace)" robot_namespace="$(arg robot_namespace)" parent_link="realsense_mountpoint"/>
+    <xacro:intel_realsense_mount prefix="camera" topic="realsense" robot_namespace="$(arg robot_namespace)" parent_link="realsense_mountpoint"/>
   </xacro:if>
   <!--
