Commit message: Added UR10 mount as a husky accessory

File: husky_description/urdf/husky.urdf.xacro (robot description, xacro)
@@ -35,4 +35,8 @@
   <xacro:arg name="realsense_rpy" default="$(optenv HUSKY_REALSENSE_RPY 0 0 0)" />
   <xacro:arg name="realsense_mount" default="$(optenv HUSKY_REALSENSE_MOUNT_FRAME sensor_arch_mount_link)" />
+  <xacro:arg name="ur10_enabled" default="$(optenv HUSKY_UR10_ENABLED 0)" />
+  <xacro:arg name="ur10_xyz" default="$(optenv HUSKY_UR10_XYZ -0.105 0.0 0)" />
+  <xacro:arg name="ur10_rpy" default="$(optenv HUSKY_UR10_RPY 0 0 3.1415927)" />
+  <xacro:arg name="ur10_mount" default="$(optenv HUSKY_UR10_MOUNT_FRAME top_plate_front_link)" />
   <xacro:property name="husky_front_bumper_extend" value="$(optenv HUSKY_FRONT_BUMPER_EXTEND 0)" />
   <xacro:property name="husky_rear_bumper_extend" value="$(optenv HUSKY_REAR_BUMPER_EXTEND 0)" />
@@ -158,5 +162,5 @@
   <xacro:if value="${sensorbar_needed_realsense or sensorbar_user_enabled or sensorbar_needed_lidar}">
     <xacro:sensor_arch prefix="" parent="top_plate_link" size="$(arg sensor_arch_height)">
-        <origin xyz="$(optenv HUSKY_SENSOR_ARCH_OFFSET 0 0 0)" rpy="$(optenv HUSKY_SENSOR_ARCH_RPY 0 0 0)"/>
+        <origin xyz="$(optenv HUSKY_SENSOR_ARCH_OFFSET -0.3 0 0)" rpy="$(optenv HUSKY_SENSOR_ARCH_RPY 0 0 0)"/>
       </xacro:sensor_arch>
   </xacro:if>
@@ -178,4 +182,14 @@
       <origin xyz="$(arg laser_3d_xyz)" rpy="$(arg laser_3d_rpy)" />
     </xacro:vlp16_mount>
+  </xacro:if>
+  <xacro:if value="$(arg ur10_enabled)">
+    <xacro:include filename="$(find husky_description)/urdf/accessories/ur10_mount.urdf.xacro"/>
+    <link name="ur10_mountpoint"/>
+    <joint name="ur10_mountpoint_joint" type="fixed">
+      <origin xyz="$(arg ur10_xyz)" rpy="$(arg ur10_rpy)" />
+      <parent link="$(arg ur10_mount)"/>
+      <child link="ur10_mountpoint" />
+    </joint>
+    <xacro:ur10_mount prefix="ur10_" use_namespace="$(arg use_namespace)" robot_namespace="$(arg robot_namespace)" parent_link="ur10_mountpoint"/>
   </xacro:if>
   <gazebo>

Commit message: update husky description to have a fake wheel

File: husky_description/urdf/husky.urdf.xacro (robot description, xacro)
@@ -47,4 +47,5 @@
   <xacro:include filename="$(find husky_description)/urdf/decorations.urdf.xacro" />
   <xacro:include filename="$(find husky_description)/urdf/wheel.urdf.xacro" />
+  <xacro:include filename="$(find husky_description)/urdf/wheel_fake.urdf.xacro" />
   <xacro:include filename="$(find husky_description)/urdf/accessories/intel_realsense.urdf.xacro"/>
   <xacro:include filename="$(find husky_description)/urdf/accessories/sick_lms1xx_mount.urdf.xacro"/>
@@ -127,4 +128,10 @@
     <origin xyz="${-wheelbase/2} ${-track/2} ${wheel_vertical_offset}" rpy="0 0 0" />
   </xacro:husky_wheel>
+  <xacro:husky_wheel_fake wheel_prefix="left_fake">
+    <origin xyz="0 ${track/2} ${wheel_vertical_offset}" rpy="0 0 0" />
+  </xacro:husky_wheel_fake>
+  <xacro:husky_wheel_fake wheel_prefix="right_fake">
+    <origin xyz="0 ${-track/2} ${wheel_vertical_offset}" rpy="0 0 0" />
+  </xacro:husky_wheel_fake>
   <xacro:husky_decorate />
   <!--

File: husky_description/urdf/wheel_fake.urdf.xacro (robot description, xacro)
@@ -21,6 +21,6 @@
 ARISING IN ANY WAY OUT OF THE USE OF THIS SOFTWARE, EVEN IF ADVISED OF THE POSSIBILITY OF SUCH DAMAGE.
 -->
-<robot xmlns:xacro="http://ros.org/wiki/xacro" name="husky_wheel">
-	<xacro:macro name="husky_wheel" params="wheel_prefix *joint_pose">
+<robot xmlns:xacro="http://ros.org/wiki/xacro" name="husky_wheel_fake">
+	<xacro:macro name="husky_wheel_fake" params="wheel_prefix *joint_pose">
 		<link name="${wheel_prefix}_wheel_link">
 			<inertial>
@@ -29,20 +29,17 @@
 				<inertia  ixx="0.02467" ixy="0" ixz="0" iyy="0.04411" iyz="0" izz="0.02467" />
 			</inertial>
-			<visual>
-				<origin xyz="0 0 0" rpy="0 0 0" />
-				<geometry>
-					<mesh filename="package://husky_description/meshes/wheel.dae" />
-				</geometry>
-			</visual>
 			<collision>
 				<origin xyz="0 0 0" rpy="${M_PI/2} 0 0" />
 				<geometry>
-					<cylinder length="${wheel_length}" radius="${wheel_radius}" />
+					<!-- <cylinder length="${wheel_length}" radius="${wheel_radius}" /> -->
+					<sphere radius="${wheel_radius}" />
 				</geometry>
 			</collision>
 		</link>
 		<gazebo reference="${wheel_prefix}_wheel_link">
-			<mu>0.0</mu>
-			<mu2>0.0</mu2>
+			<mu>100.0</mu>
+			<mu2>100.0</mu2>
+			<kp>10000000.0</kp>
+    	<kd>1.0</kd>
 		</gazebo>
 		<joint name="${wheel_prefix}_wheel" type="continuous">

Commit message: remove fake wheel, and change physics constants in wheel link

File: husky_description/urdf/husky.urdf.xacro (robot description, xacro)
@@ -47,5 +47,4 @@
   <xacro:include filename="$(find husky_description)/urdf/decorations.urdf.xacro" />
   <xacro:include filename="$(find husky_description)/urdf/wheel.urdf.xacro" />
-  <xacro:include filename="$(find husky_description)/urdf/wheel_fake.urdf.xacro" />
   <xacro:include filename="$(find husky_description)/urdf/accessories/intel_realsense.urdf.xacro"/>
   <xacro:include filename="$(find husky_description)/urdf/accessories/sick_lms1xx_mount.urdf.xacro"/>
@@ -128,10 +127,4 @@
     <origin xyz="${-wheelbase/2} ${-track/2} ${wheel_vertical_offset}" rpy="0 0 0" />
   </xacro:husky_wheel>
-  <xacro:husky_wheel_fake wheel_prefix="left_fake">
-    <origin xyz="0 ${track/2} ${wheel_vertical_offset}" rpy="0 0 0" />
-  </xacro:husky_wheel_fake>
-  <xacro:husky_wheel_fake wheel_prefix="right_fake">
-    <origin xyz="0 ${-track/2} ${wheel_vertical_offset}" rpy="0 0 0" />
-  </xacro:husky_wheel_fake>
   <xacro:husky_decorate />
   <!--

File: husky_description/urdf/wheel.urdf.xacro (robot description, xacro)
@@ -43,6 +43,9 @@
 		</link>
 		<gazebo reference="${wheel_prefix}_wheel_link">
-			<mu1>0.0</mu1>
-			<mu2>0.0</mu2>
+			<mu1 value="100.0"/>
+			<mu2 value="100.0"/>
+			<kp value="10000000.0" />
+			<kd value="1.0" />
+			<!-- <fdir1 value="1 0 0"/> -->  <!-- Directional Friction is broken (https://github.com/gazebosim/gazebo-classic/issues/2068) -->
 		</gazebo>
 		<joint name="${wheel_prefix}_wheel" type="continuous">
